Commit message: Updated weights to be reflective of 1/4th inch aluminium plates for the main plates and the ebox, updated the arm to have 1/8th inch aluminium weights, updated the claw and the thrusters to have plastic weights

File: src/rov_description/urdf/rov.xacro (robot description, xacro)
@@ -7,5 +7,5 @@
   <inertial>
     <origin xyz="-0.00884973146778553 -0.2071832362580056 0.0001594860889622284" rpy="0 0 0"/>
-    <mass value="3.285705148468138"/>
+    <mass value="3.294247"/>
     <inertia ixx="0.151251" iyy="0.28825" izz="0.137021" ixy="0.0" iyz="-0.0" ixz="6.7e-05"/>
   </inertial>
@@ -27,5 +27,5 @@
   <inertial>
     <origin xyz="-0.00449028432226567 0.1047212706889887 -0.004490284322260396" rpy="0 0 0"/>
-    <mass value="0.34092339371935965"/>
+    <mass value="0.341030"/>
     <inertia ixx="0.001286" iyy="7.1e-05" izz="0.001286" ixy="0.0" iyz="0.0" ixz="3.1e-05"/>
   </inertial>
@@ -47,5 +47,5 @@
   <inertial>
     <origin xyz="0.004490284322265392 0.1047212706889887 -0.004490284322267224" rpy="0 0 0"/>
-    <mass value="0.34092339371935965"/>
+    <mass value="0.341030"/>
     <inertia ixx="0.001286" iyy="7.1e-05" izz="0.001286" ixy="-0.0" iyz="0.0" ixz="-3.1e-05"/>
   </inertial>
@@ -67,5 +67,5 @@
   <inertial>
     <origin xyz="0.004490284322271526 0.10472127068898884 0.004490284322263699" rpy="0 0 0"/>
-    <mass value="0.34092339371935965"/>
+    <mass value="0.341030"/>
     <inertia ixx="0.001286" iyy="7.1e-05" izz="0.001286" ixy="-0.0" iyz="-0.0" ixz="3.1e-05"/>
   </inertial>
@@ -87,5 +87,5 @@
   <inertial>
     <origin xyz="-0.004490284322259119 0.10472127068898884 0.004490284322270055" rpy="0 0 0"/>
-    <mass value="0.34092339371935965"/>
+    <mass value="0.341030"/>
     <inertia ixx="0.001286" iyy="7.1e-05" izz="0.001286" ixy="0.0" iyz="-0.0" ixz="-3.1e-05"/>
   </inertial>
@@ -107,5 +107,5 @@
   <inertial>
     <origin xyz="-0.08600000000000418 0.023514887456752447 0.0" rpy="0 0 0"/>
-    <mass value="0.09679089766266749"/>
+    <mass value="0.237318"/>
     <inertia ixx="3.9e-05" iyy="0.000228" izz="0.000264" ixy="-0.0" iyz="0.0" ixz="-0.0"/>
   </inertial>
@@ -127,5 +127,5 @@
   <inertial>
     <origin xyz="-0.08600000000000434 0.023514887456752447 0.0" rpy="0 0 0"/>
-    <mass value="0.09679089766266749"/>
+    <mass value="0.237318"/>
     <inertia ixx="3.9e-05" iyy="0.000228" izz="0.000264" ixy="-0.0" iyz="0.0" ixz="-0.0"/>
   </inertial>
@@ -147,5 +147,5 @@
   <inertial>
     <origin xyz="-0.012365898764221173 -3.2044554445498363e-06 -0.012368635677551754" rpy="0 0 0"/>
-    <mass value="0.008326303172342044"/>
+    <mass value="0.008653"/>
     <inertia ixx="3e-06" iyy="2e-06" izz="3e-06" ixy="0.0" iyz="-0.0" ixz="1e-06"/>
   </inertial>
@@ -167,5 +167,5 @@
   <inertial>
     <origin xyz="-0.01236878771037464 -3.2044554437726802e-06 0.012365746731409555" rpy="0 0 0"/>
-    <mass value="0.008326303172342044"/>
+    <mass value="0.008653"/>
     <inertia ixx="3e-06" iyy="2e-06" izz="3e-06" ixy="-0.0" iyz="-0.0" ixz="-1e-06"/>
   </inertial>
@@ -187,5 +187,5 @@
   <inertial>
     <origin xyz="0.012365898764223893 -3.2044554439669692e-06 0.012368635677550976" rpy="0 0 0"/>
-    <mass value="0.008326303172342044"/>
+    <mass value="0.008653"/>
     <inertia ixx="3e-06" iyy="2e-06" izz="3e-06" ixy="-0.0" iyz="0.0" ixz="1e-06"/>
   </inertial>
@@ -207,5 +207,5 @@
   <inertial>
     <origin xyz="0.012368787710376472 -3.204455443467369e-06 -0.012365746731402838" rpy="0 0 0"/>
-    <mass value="0.008326303172342044"/>
+    <mass value="0.008653"/>
     <inertia ixx="3e-06" iyy="2e-06" izz="3e-06" ixy="0.0" iyz="0.0" ixz="-1e-06"/>
   </inertial>
@@ -227,5 +227,5 @@
   <inertial>
     <origin xyz="4.065704311606577e-06 0.017490034130872245 -4.6608003942405496e-07" rpy="0 0 0"/>
-    <mass value="0.008326303172342044"/>
+    <mass value="0.008653"/>
     <inertia ixx="2e-06" iyy="3e-06" izz="2e-06" ixy="-0.0" iyz="0.0" ixz="0.0"/>
   </inertial>
@@ -247,5 +247,5 @@
   <inertial>
     <origin xyz="4.065704307693041e-06 0.01749003413087242 -1.1767581619970269e-06" rpy="0 0 0"/>
-    <mass value="0.008326303172342044"/>
+    <mass value="0.008653"/>
     <inertia ixx="2e-06" iyy="3e-06" izz="2e-06" ixy="-0.0" iyz="0.0" ixz="0.0"/>
   </inertial>
@@ -267,5 +267,5 @@
   <inertial>
     <origin xyz="3.3550261890058497e-06 0.01749003413087237 -1.176758154003421e-06" rpy="0 0 0"/>
-    <mass value="0.008326303172342044"/>
+    <mass value="0.008653"/>
     <inertia ixx="2e-06" iyy="3e-06" izz="2e-06" ixy="-0.0" iyz="0.0" ixz="0.0"/>
   </inertial>
@@ -287,5 +287,5 @@
   <inertial>
     <origin xyz="3.3550261931969416e-06 0.017490034130872203 -4.660800397293663e-07" rpy="0 0 0"/>
-    <mass value="0.008326303172342044"/>
+    <mass value="0.008653"/>
     <inertia ixx="2e-06" iyy="3e-06" izz="2e-06" ixy="-0.0" iyz="0.0" ixz="0.0"/>
   </inertial>
@@ -307,5 +307,5 @@
   <inertial>
     <origin xyz="0.1419635000000286 0.08575276315482112 0.12499300000000114" rpy="0 0 0"/>
-    <mass value="2.95500253978019"/>
+    <mass value="7.975075"/>
     <inertia ixx="0.034054" iyy="0.049082" izz="0.034054" ixy="0.0" iyz="-0.0" ixz="-0.0"/>
   </inertial>
@@ -327,5 +327,5 @@
   <inertial>
     <origin xyz="-0.04500000000000731 0.09562846640758502 -4.999999958441026e-07" rpy="0 0 0"/>
-    <mass value="0.19465175506780696"/>
+    <mass value="0.194902"/>
     <inertia ixx="0.000871" iyy="0.000269" izz="0.001138" ixy="0.0" iyz="-0.0" ixz="-0.0"/>
   </inertial>
@@ -347,5 +347,5 @@
   <inertial>
     <origin xyz="-0.04500000000000837 0.09562846640758497 -4.999999957469581e-07" rpy="0 0 0"/>
-    <mass value="0.19465175506780696"/>
+    <mass value="0.194902"/>
     <inertia ixx="0.000871" iyy="0.000269" izz="0.001138" ixy="0.0" iyz="0.0" ixz="-0.0"/>
   </inertial>
@@ -367,5 +367,5 @@
   <inertial>
     <origin xyz="-0.016000000000067904 -0.025999999999988116 0.004395257122678596" rpy="0 0 0"/>
-    <mass value="0.014289632808758179"/>
+    <mass value="0.038613"/>
     <inertia ixx="8e-06" iyy="5e-06" izz="1.2e-05" ixy="-0.0" iyz="-0.0" ixz="-0.0"/>
   </inertial>
@@ -387,5 +387,5 @@
   <inertial>
     <origin xyz="0.016000000000073955 -0.0259999999999882 -0.004396257122670222" rpy="0 0 0"/>
-    <mass value="0.014289632808758179"/>
+    <mass value="0.038613"/>
     <inertia ixx="8e-06" iyy="5e-06" izz="1.2e-05" ixy="0.0" iyz="0.0" ixz="-0.0"/>
   </inertial>
@@ -407,5 +407,5 @@
   <inertial>
     <origin xyz="5.525922222582302e-07 -0.07493659975726129 5.001667301232637e-07" rpy="0 0 0"/>
-    <mass value="0.031662848727866975"/>
+    <mass value="0.085598"/>
     <inertia ixx="7.3e-05" iyy="1.6e-05" izz="8.9e-05" ixy="0.0" iyz="-0.0" ixz="0.0"/>
   </inertial>
@@ -427,5 +427,5 @@
   <inertial>
     <origin xyz="-0.09414946806162938 6.653102950542056e-05 0.002887254879548433" rpy="0 0 0"/>
-    <mass value="0.23816081829076916"/>
+    <mass value="0.238329"/>
     <inertia ixx="0.000253" iyy="0.002317" izz="0.00222" ixy="0.0" iyz="-1e-06" ixz="1e-06"/>
   </inertial>
@@ -447,5 +447,5 @@
   <inertial>
     <origin xyz="0.036504021537288295 0.0010587831807864073 0.024711763155022364" rpy="0 0 0"/>
-    <mass value="0.038521930758269235"/>
+    <mass value="0.104132"/>
     <inertia ixx="2.9e-05" iyy="4e-05" izz="3.9e-05" ixy="-2e-06" iyz="0.0" ixz="0.0"/>
   </inertial>
@@ -467,5 +467,5 @@
   <inertial>
     <origin xyz="0.020570162349985127 0.0008209490871033537 -8.376397228182769e-05" rpy="0 0 0"/>
-    <mass value="0.016346422343594975"/>
+    <mass value="0.044156"/>
     <inertia ixx="4e-06" iyy="7e-06" izz="5e-06" ixy="-0.0" iyz="0.0" ixz="0.0"/>
   </inertial>
@@ -487,5 +487,5 @@
   <inertial>
     <origin xyz="0.08354760410561307 -0.005972879878576573 -0.010043597389812697" rpy="0 0 0"/>
-    <mass value="0.08375835449631712"/>
+    <mass value="0.032267"/>
     <inertia ixx="1.3e-05" iyy="0.000195" izz="0.00019" ixy="-0.0" iyz="0.0" ixz="-6e-06"/>
   </inertial>
@@ -507,5 +507,5 @@
   <inertial>
     <origin xyz="0.07566774937988974 -0.0059640260689888674 0.009495558359122119" rpy="0 0 0"/>
-    <mass value="0.07927492984287204"/>
+    <mass value="0.030533"/>
     <inertia ixx="1.2e-05" iyy="0.000193" izz="0.000188" ixy="0.0" iyz="-0.0" ixz="4e-06"/>
   </inertial>
@@ -547,5 +547,5 @@
   <inertial>
     <origin xyz="0.24782424120968954 0.00016204304487000198 -0.2467838984061316" rpy="0 0 0"/>
-    <mass value="3.2351726296403394"/>
+    <mass value="3.242845"/>
     <inertia ixx="0.166436" iyy="0.317863" izz="0.151449" ixy="-1.4e-05" iyz="-5e-06" ixz="-0.001482"/>
   </inertial>
@@ -567,5 +567,5 @@
   <inertial>
     <origin xyz="-0.02684279690594965 -0.00950557626176958 0.041487649225129264" rpy="0 0 0"/>
-    <mass value="0.15065662889769457"/>
+    <mass value="0.156158"/>
     <inertia ixx="0.000156" iyy="0.000141" izz="0.000154" ixy="0.0" iyz="0.0" ixz="1.8e-05"/>
   </inertial>
@@ -587,5 +587,5 @@
   <inertial>
     <origin xyz="0.03416973472258347 -0.019855474384367508 -0.03416184869756059" rpy="0 0 0"/>
-    <mass value="0.15065662889769457"/>
+    <mass value="0.156158"/>
     <inertia ixx="0.000139" iyy="0.000173" izz="0.000139" ixy="1e-06" iyz="-1e-06" ixz="2e-06"/>
   </inertial>
@@ -607,5 +607,5 @@
   <inertial>
     <origin xyz="0.026842796905951205 -0.009494423738229812 0.04148764922513448" rpy="0 0 0"/>
-    <mass value="0.15065662889769457"/>
+    <mass value="0.156158"/>
     <inertia ixx="0.000156" iyy="0.000141" izz="0.000154" ixy="0.0" iyz="-0.0" ixz="-1.8e-05"/>
   </inertial>
@@ -627,5 +627,5 @@
   <inertial>
     <origin xyz="-0.03416184869755892 -0.019855474384367487 -0.03416973472257842" rpy="0 0 0"/>
-    <mass value="0.15065662889769457"/>
+    <mass value="0.156158"/>
     <inertia ixx="0.000139" iyy="0.000173" izz="0.000139" ixy="-1e-06" iyz="-1e-06" ixz="-2e-06"/>
   </inertial>
@@ -647,5 +647,5 @@
   <inertial>
     <origin xyz="0.026842796905956756 -0.009505576261768914 -0.041487649225126155" rpy="0 0 0"/>
-    <mass value="0.15065662889769457"/>
+    <mass value="0.156158"/>
     <inertia ixx="0.000156" iyy="0.000141" izz="0.000154" ixy="-0.0" iyz="-0.0" ixz="1.8e-05"/>
   </inertial>
@@ -667,5 +667,5 @@
   <inertial>
     <origin xyz="-0.03416973472257784 -0.019855474384367307 0.034161848697562724" rpy="0 0 0"/>
-    <mass value="0.15065662889769457"/>
+    <mass value="0.156158"/>
     <inertia ixx="0.000139" iyy="0.000173" izz="0.000139" ixy="-1e-06" iyz="1e-06" ixz="2e-06"/>
   </inertial>
@@ -687,5 +687,5 @@
   <inertial>
     <origin xyz="-0.0268427969059446 -0.009494423738229896 -0.04148764922513154" rpy="0 0 0"/>
-    <mass value="0.15065662889769457"/>
+    <mass value="0.156158"/>
     <inertia ixx="0.000156" iyy="0.000141" izz="0.000154" ixy="-0.0" iyz="0.0" ixz="-1.8e-05"/>
   </inertial>
@@ -707,5 +707,5 @@
   <inertial>
     <origin xyz="0.034161848697564196 -0.019855474384367335 0.03416973472258247" rpy="0 0 0"/>
-    <mass value="0.15065662889769457"/>
+    <mass value="0.156158"/>
     <inertia ixx="0.000139" iyy="0.000173" izz="0.000139" ixy="1e-06" iyz="1e-06" ixz="-2e-06"/>
   </inertial>

Commit message: Edited zero of shoulder and elbow joint to be more accurate

File: src/rov_description/urdf/rov.xacro (robot description, xacro)
@@ -833,5 +833,5 @@
 </joint>
 <joint name="shoulderjoint" type="continuous">
-  <origin xyz="0.0 -0.102 -0.003175" rpy="0 0 0"/>
+  <origin xyz="0.0 -0.102 -0.003175" rpy="0 0 3.141592653589793"/>
   <parent link="V4B_SupportPlate_v1_1"/>
   <child link="shoulder_1"/>
@@ -839,5 +839,5 @@
 </joint>
 <joint name="elbowjoint" type="continuous">
-  <origin xyz="-0.2075 0.0 -0.004174" rpy="0 0 0"/>
+  <origin xyz="-0.2075 0.0 -0.004174" rpy="0 0 -3.141592653589793"/>
   <parent link="shoulder_1"/>
   <child link="elbow_1"/>

Commit message: Edited launch file to properly parse xacro as xacro and not yaml, edited plugins to work with SBRT's Repo, the gazebo was edited to prevent the display erroes, the urdf was edited to fix the collision meshes

File: src/rov_description/urdf/rov.xacro (robot description, xacro)
@@ -20,5 +20,5 @@
     <origin xyz="0 0 0" rpy="0 0 0"/>
     <geometry>
-      <mesh filename="file://$(find rov_description)/meshes/base_link.stl" scale="0.001 0.001 0.001"/>
+      <box size="0.6 0.4 0.25"/>
     </geometry>
   </collision>
