Commit message: Redid simulation for the MATE-ROV 2026 with the updated arm

File: src/rov_description/urdf/rov.xacro (robot description, xacro)
@@ -6,7 +6,7 @@
 <link name="base_link">
   <inertial>
-    <origin xyz="-0.00884973146778553 -0.2071832362580056 0.0001594860889622284" rpy="0 0 0"/>
-    <mass value="3.294247"/>
-    <inertia ixx="0.151251" iyy="0.28825" izz="0.137021" ixy="0.0" iyz="-0.0" ixz="6.7e-05"/>
+    <origin xyz="-5.6904454281479577e-05 0.002259535915373094 -0.055056343609268456" rpy="0 0 0"/>
+    <mass value="2.647880364444541"/>
+    <inertia ixx="0.097024" iyy="0.140548" izz="0.237555" ixy="-1.6e-05" iyz="-0.0" ixz="-0.0"/>
   </inertial>
   <visual>
@@ -20,285 +20,765 @@
     <origin xyz="0 0 0" rpy="0 0 0"/>
     <geometry>
-      <box size="0.6 0.4 0.25"/>
-    </geometry>
-  </collision>
-</link>
-<link name="VerticalThrusterSupportBeams_2">
-  <inertial>
-    <origin xyz="-0.00449028432226567 0.1047212706889887 -0.004490284322260396" rpy="0 0 0"/>
-    <mass value="0.341030"/>
-    <inertia ixx="0.001286" iyy="7.1e-05" izz="0.001286" ixy="0.0" iyz="0.0" ixz="3.1e-05"/>
-  </inertial>
-  <visual>
-    <origin xyz="-0.243664 0.207 -0.243664" rpy="0 0 0"/>
-    <geometry>
-      <mesh filename="file://$(find rov_description)/meshes/VerticalThrusterSupportBeams_2.stl" scale="0.001 0.001 0.001"/>
-    </geometry>
-    <material name="silver"/>
-  </visual>
-  <collision>
-    <origin xyz="-0.243664 0.207 -0.243664" rpy="0 0 0"/>
-    <geometry>
-      <mesh filename="file://$(find rov_description)/meshes/VerticalThrusterSupportBeams_2.stl" scale="0.001 0.001 0.001"/>
-    </geometry>
-  </collision>
-</link>
-<link name="VerticalThrusterSupportBeams_1">
-  <inertial>
-    <origin xyz="0.004490284322265392 0.1047212706889887 -0.004490284322267224" rpy="0 0 0"/>
-    <mass value="0.341030"/>
-    <inertia ixx="0.001286" iyy="7.1e-05" izz="0.001286" ixy="-0.0" iyz="0.0" ixz="-3.1e-05"/>
-  </inertial>
-  <visual>
-    <origin xyz="0.243664 0.207 -0.243664" rpy="0 0 0"/>
-    <geometry>
-      <mesh filename="file://$(find rov_description)/meshes/VerticalThrusterSupportBeams_1.stl" scale="0.001 0.001 0.001"/>
-    </geometry>
-    <material name="silver"/>
-  </visual>
-  <collision>
-    <origin xyz="0.243664 0.207 -0.243664" rpy="0 0 0"/>
-    <geometry>
-      <mesh filename="file://$(find rov_description)/meshes/VerticalThrusterSupportBeams_1.stl" scale="0.001 0.001 0.001"/>
-    </geometry>
-  </collision>
-</link>
-<link name="VerticalThrusterSupportBeams_4">
-  <inertial>
-    <origin xyz="0.004490284322271526 0.10472127068898884 0.004490284322263699" rpy="0 0 0"/>
-    <mass value="0.341030"/>
-    <inertia ixx="0.001286" iyy="7.1e-05" izz="0.001286" ixy="-0.0" iyz="-0.0" ixz="3.1e-05"/>
-  </inertial>
-  <visual>
-    <origin xyz="0.243664 0.207 0.243664" rpy="0 0 0"/>
-    <geometry>
-      <mesh filename="file://$(find rov_description)/meshes/VerticalThrusterSupportBeams_4.stl" scale="0.001 0.001 0.001"/>
-    </geometry>
-    <material name="silver"/>
-  </visual>
-  <collision>
-    <origin xyz="0.243664 0.207 0.243664" rpy="0 0 0"/>
-    <geometry>
-      <mesh filename="file://$(find rov_description)/meshes/VerticalThrusterSupportBeams_4.stl" scale="0.001 0.001 0.001"/>
-    </geometry>
-  </collision>
-</link>
-<link name="VerticalThrusterSupportBeams_3">
-  <inertial>
-    <origin xyz="-0.004490284322259119 0.10472127068898884 0.004490284322270055" rpy="0 0 0"/>
-    <mass value="0.341030"/>
-    <inertia ixx="0.001286" iyy="7.1e-05" izz="0.001286" ixy="0.0" iyz="-0.0" ixz="-3.1e-05"/>
-  </inertial>
-  <visual>
-    <origin xyz="-0.243664 0.207 0.243664" rpy="0 0 0"/>
-    <geometry>
-      <mesh filename="file://$(find rov_description)/meshes/VerticalThrusterSupportBeams_3.stl" scale="0.001 0.001 0.001"/>
-    </geometry>
-    <material name="silver"/>
-  </visual>
-  <collision>
-    <origin xyz="-0.243664 0.207 0.243664" rpy="0 0 0"/>
-    <geometry>
-      <mesh filename="file://$(find rov_description)/meshes/VerticalThrusterSupportBeams_3.stl" scale="0.001 0.001 0.001"/>
-    </geometry>
-  </collision>
-</link>
-<link name="Handles_2">
-  <inertial>
-    <origin xyz="-0.08600000000000418 0.023514887456752447 0.0" rpy="0 0 0"/>
-    <mass value="0.237318"/>
-    <inertia ixx="3.9e-05" iyy="0.000228" izz="0.000264" ixy="-0.0" iyz="0.0" ixz="-0.0"/>
-  </inertial>
-  <visual>
-    <origin xyz="-0.086 -0.00635 0.318" rpy="0 0 0"/>
-    <geometry>
-      <mesh filename="file://$(find rov_description)/meshes/Handles_2.stl" scale="0.001 0.001 0.001"/>
-    </geometry>
-    <material name="silver"/>
-  </visual>
-  <collision>
-    <origin xyz="-0.086 -0.00635 0.318" rpy="0 0 0"/>
-    <geometry>
-      <mesh filename="file://$(find rov_description)/meshes/Handles_2.stl" scale="0.001 0.001 0.001"/>
-    </geometry>
-  </collision>
-</link>
-<link name="Handles_1">
-  <inertial>
-    <origin xyz="-0.08600000000000434 0.023514887456752447 0.0" rpy="0 0 0"/>
-    <mass value="0.237318"/>
-    <inertia ixx="3.9e-05" iyy="0.000228" izz="0.000264" ixy="-0.0" iyz="0.0" ixz="-0.0"/>
-  </inertial>
-  <visual>
-    <origin xyz="-0.086 -0.00635 -0.318" rpy="0 0 0"/>
-    <geometry>
-      <mesh filename="file://$(find rov_description)/meshes/Handles_1.stl" scale="0.001 0.001 0.001"/>
-    </geometry>
-    <material name="silver"/>
-  </visual>
-  <collision>
-    <origin xyz="-0.086 -0.00635 -0.318" rpy="0 0 0"/>
-    <geometry>
-      <mesh filename="file://$(find rov_description)/meshes/Handles_1.stl" scale="0.001 0.001 0.001"/>
-    </geometry>
-  </collision>
-</link>
-<link name="propbackright_1">
-  <inertial>
-    <origin xyz="-0.012365898764221173 -3.2044554445498363e-06 -0.012368635677551754" rpy="0 0 0"/>
-    <mass value="0.008653"/>
-    <inertia ixx="3e-06" iyy="2e-06" izz="3e-06" ixy="0.0" iyz="-0.0" ixz="1e-06"/>
-  </inertial>
-  <visual>
-    <origin xyz="0.25586 0.102 -0.300764" rpy="0 0 0"/>
-    <geometry>
-      <mesh filename="file://$(find rov_description)/meshes/propbackright_1.stl" scale="0.001 0.001 0.001"/>
-    </geometry>
-    <material name="silver"/>
-  </visual>
-  <collision>
-    <origin xyz="0.25586 0.102 -0.300764" rpy="0 0 0"/>
-    <geometry>
-      <mesh filename="file://$(find rov_description)/meshes/propbackright_1.stl" scale="0.001 0.001 0.001"/>
-    </geometry>
-  </collision>
-</link>
-<link name="propbackleft_1">
-  <inertial>
-    <origin xyz="-0.01236878771037464 -3.2044554437726802e-06 0.012365746731409555" rpy="0 0 0"/>
-    <mass value="0.008653"/>
-    <inertia ixx="3e-06" iyy="2e-06" izz="3e-06" ixy="-0.0" iyz="-0.0" ixz="-1e-06"/>
-  </inertial>
-  <visual>
-    <origin xyz="0.25586 0.102 0.300764" rpy="0 0 0"/>
-    <geometry>
-      <mesh filename="file://$(find rov_description)/meshes/propbackleft_1.stl" scale="0.001 0.001 0.001"/>
-    </geometry>
-    <material name="silver"/>
-  </visual>
-  <collision>
-    <origin xyz="0.25586 0.102 0.300764" rpy="0 0 0"/>
-    <geometry>
-      <mesh filename="file://$(find rov_description)/meshes/propbackleft_1.stl" scale="0.001 0.001 0.001"/>
-    </geometry>
-  </collision>
-</link>
-<link name="propfrontleft_1">
-  <inertial>
-    <origin xyz="0.012365898764223893 -3.2044554439669692e-06 0.012368635677550976" rpy="0 0 0"/>
-    <mass value="0.008653"/>
-    <inertia ixx="3e-06" iyy="2e-06" izz="3e-06" ixy="-0.0" iyz="0.0" ixz="1e-06"/>
-  </inertial>
-  <visual>
-    <origin xyz="-0.25586 0.102 0.300764" rpy="0 0 0"/>
-    <geometry>
-      <mesh filename="file://$(find rov_description)/meshes/propfrontleft_1.stl" scale="0.001 0.001 0.001"/>
-    </geometry>
-    <material name="silver"/>
-  </visual>
-  <collision>
-    <origin xyz="-0.25586 0.102 0.300764" rpy="0 0 0"/>
-    <geometry>
-      <mesh filename="file://$(find rov_description)/meshes/propfrontleft_1.stl" scale="0.001 0.001 0.001"/>
-    </geometry>
-  </collision>
-</link>
-<link name="propfrontright_1">
-  <inertial>
-    <origin xyz="0.012368787710376472 -3.204455443467369e-06 -0.012365746731402838" rpy="0 0 0"/>
-    <mass value="0.008653"/>
-    <inertia ixx="3e-06" iyy="2e-06" izz="3e-06" ixy="0.0" iyz="0.0" ixz="-1e-06"/>
-  </inertial>
-  <visual>
-    <origin xyz="-0.25586 0.102 -0.300764" rpy="0 0 0"/>
-    <geometry>
-      <mesh filename="file://$(find rov_description)/meshes/propfrontright_1.stl" scale="0.001 0.001 0.001"/>
-    </geometry>
-    <material name="silver"/>
-  </visual>
-  <collision>
-    <origin xyz="-0.25586 0.102 -0.300764" rpy="0 0 0"/>
-    <geometry>
-      <mesh filename="file://$(find rov_description)/meshes/propfrontright_1.stl" scale="0.001 0.001 0.001"/>
-    </geometry>
-  </collision>
-</link>
-<link name="proptopfrontright_1">
-  <inertial>
-    <origin xyz="4.065704311606577e-06 0.017490034130872245 -4.6608003942405496e-07" rpy="0 0 0"/>
-    <mass value="0.008653"/>
-    <inertia ixx="2e-06" iyy="3e-06" izz="2e-06" ixy="-0.0" iyz="0.0" ixz="0.0"/>
-  </inertial>
-  <visual>
-    <origin xyz="-0.200035 0.076752 -0.200035" rpy="0 0 0"/>
-    <geometry>
-      <mesh filename="file://$(find rov_description)/meshes/proptopfrontright_1.stl" scale="0.001 0.001 0.001"/>
-    </geometry>
-    <material name="silver"/>
-  </visual>
-  <collision>
-    <origin xyz="-0.200035 0.076752 -0.200035" rpy="0 0 0"/>
-    <geometry>
-      <mesh filename="file://$(find rov_description)/meshes/proptopfrontright_1.stl" scale="0.001 0.001 0.001"/>
-    </geometry>
-  </collision>
-</link>
-<link name="proptopfrontleft_1">
-  <inertial>
-    <origin xyz="4.065704307693041e-06 0.01749003413087242 -1.1767581619970269e-06" rpy="0 0 0"/>
-    <mass value="0.008653"/>
-    <inertia ixx="2e-06" iyy="3e-06" izz="2e-06" ixy="-0.0" iyz="0.0" ixz="0.0"/>
-  </inertial>
-  <visual>
-    <origin xyz="-0.200035 0.076752 0.200035" rpy="0 0 0"/>
-    <geometry>
-      <mesh filename="file://$(find rov_description)/meshes/proptopfrontleft_1.stl" scale="0.001 0.001 0.001"/>
-    </geometry>
-    <material name="silver"/>
-  </visual>
-  <collision>
-    <origin xyz="-0.200035 0.076752 0.200035" rpy="0 0 0"/>
-    <geometry>
-      <mesh filename="file://$(find rov_description)/meshes/proptopfrontleft_1.stl" scale="0.001 0.001 0.001"/>
-    </geometry>
-  </collision>
-</link>
-<link name="proptopbackleft_1">
-  <inertial>
-    <origin xyz="3.3550261890058497e-06 0.01749003413087237 -1.176758154003421e-06" rpy="0 0 0"/>
-    <mass value="0.008653"/>
-    <inertia ixx="2e-06" iyy="3e-06" izz="2e-06" ixy="-0.0" iyz="0.0" ixz="0.0"/>
-  </inertial>
-  <visual>
-    <origin xyz="0.200035 0.076752 0.200035" rpy="0 0 0"/>
-    <geometry>
-      <mesh filename="file://$(find rov_description)/meshes/proptopbackleft_1.stl" scale="0.001 0.001 0.001"/>
-    </geometry>
-    <material name="silver"/>
-  </visual>
-  <collision>
-    <origin xyz="0.200035 0.076752 0.200035" rpy="0 0 0"/>
-    <geometry>
-      <mesh filename="file://$(find rov_description)/meshes/proptopbackleft_1.stl" scale="0.001 0.001 0.001"/>
-    </geometry>
-  </collision>
-</link>
-<link name="proptopbackright_1">
-  <inertial>
-    <origin xyz="3.3550261931969416e-06 0.017490034130872203 -4.660800397293663e-07" rpy="0 0 0"/>
-    <mass value="0.008653"/>
-    <inertia ixx="2e-06" iyy="3e-06" izz="2e-06" ixy="-0.0" iyz="0.0" ixz="0.0"/>
-  </inertial>
-  <visual>
-    <origin xyz="0.200035 0.076752 -0.200035" rpy="0 0 0"/>
-    <geometry>
-      <mesh filename="file://$(find rov_description)/meshes/proptopbackright_1.stl" scale="0.001 0.001 0.001"/>
-    </geometry>
-    <material name="silver"/>
-  </visual>
-  <collision>
-    <origin xyz="0.200035 0.076752 -0.200035" rpy="0 0 0"/>
-    <geometry>
-      <mesh filename="file://$(find rov_description)/meshes/proptopbackright_1.stl" scale="0.001 0.001 0.001"/>
+      <mesh filename="file://$(find rov_description)/meshes/base_link.stl" scale="0.001 0.001 0.001"/>
+    </geometry>
+  </collision>
+</link>
+<link name="VerticalThrusterBeams_V7_v1__3__1">
+  <inertial>
+    <origin xyz="0.016970218305073115 -0.016970173279726886 0.11591472778502045" rpy="0 0 0"/>
+    <mass value="0.20947204476435513"/>
+    <inertia ixx="0.000871" iyy="0.000871" izz="4.9e-05" ixy="2.2e-05" iyz="-0.0" ixz="-0.0"/>
+  </inertial>
+  <visual>
+    <origin xyz="0.28025 0.301231 0.054378" rpy="0 0 0"/>
+    <geometry>
+      <mesh filename="file://$(find rov_description)/meshes/VerticalThrusterBeams_V7_v1__3__1.stl" scale="0.001 0.001 0.001"/>
+    </geometry>
+    <material name="silver"/>
+  </visual>
+  <collision>
+    <origin xyz="0.28025 0.301231 0.054378" rpy="0 0 0"/>
+    <geometry>
+      <mesh filename="file://$(find rov_description)/meshes/VerticalThrusterBeams_V7_v1__3__1.stl" scale="0.001 0.001 0.001"/>
+    </geometry>
+  </collision>
+</link>
+<link name="VerticalThrusterBeams_V7_v1__2__1">
+  <inertial>
+    <origin xyz="0.01697021830510126 0.01697054739762352 0.11591472778502315" rpy="0 0 0"/>
+    <mass value="0.20947204476435513"/>
+    <inertia ixx="0.000871" iyy="0.000871" izz="4.9e-05" ixy="-2.2e-05" iyz="0.0" ixz="-0.0"/>
+  </inertial>
+  <visual>
+    <origin xyz="0.28025 -0.191105 0.054378" rpy="0 0 0"/>
+    <geometry>
+      <mesh filename="file://$(find rov_description)/meshes/VerticalThrusterBeams_V7_v1__2__1.stl" scale="0.001 0.001 0.001"/>
+    </geometry>
+    <material name="silver"/>
+  </visual>
+  <collision>
+    <origin xyz="0.28025 -0.191105 0.054378" rpy="0 0 0"/>
+    <geometry>
+      <mesh filename="file://$(find rov_description)/meshes/VerticalThrusterBeams_V7_v1__2__1.stl" scale="0.001 0.001 0.001"/>
+    </geometry>
+  </collision>
+</link>
+<link name="VerticalThrusterBeams_V7_v1_1">
+  <inertial>
+    <origin xyz="0.016970360338689428 -0.016971031246166945 0.11591472778502301" rpy="0 0 0"/>
+    <mass value="0.20947204476435513"/>
+    <inertia ixx="0.000871" iyy="0.000871" izz="4.9e-05" ixy="2.2e-05" iyz="0.0" ixz="0.0"/>
+  </inertial>
+  <visual>
+    <origin xyz="-0.246168 -0.225188 0.054378" rpy="0 0 0"/>
+    <geometry>
+      <mesh filename="file://$(find rov_description)/meshes/VerticalThrusterBeams_V7_v1_1.stl" scale="0.001 0.001 0.001"/>
+    </geometry>
+    <material name="silver"/>
+  </visual>
+  <collision>
+    <origin xyz="-0.246168 -0.225188 0.054378" rpy="0 0 0"/>
+    <geometry>
+      <mesh filename="file://$(find rov_description)/meshes/VerticalThrusterBeams_V7_v1_1.stl" scale="0.001 0.001 0.001"/>
+    </geometry>
+  </collision>
+</link>
+<link name="VerticalThrusterBeams_V7_v1__1__1">
+  <inertial>
+    <origin xyz="0.01697036033866145 0.01697040536400729 0.11591472778502049" rpy="0 0 0"/>
+    <mass value="0.20947204476435513"/>
+    <inertia ixx="0.000871" iyy="0.000871" izz="4.9e-05" ixy="-2.2e-05" iyz="-0.0" ixz="0.0"/>
+  </inertial>
+  <visual>
+    <origin xyz="-0.246168 0.335313 0.054378" rpy="0 0 0"/>
+    <geometry>
+      <mesh filename="file://$(find rov_description)/meshes/VerticalThrusterBeams_V7_v1__1__1.stl" scale="0.001 0.001 0.001"/>
+    </geometry>
+    <material name="silver"/>
+  </visual>
+  <collision>
+    <origin xyz="-0.246168 0.335313 0.054378" rpy="0 0 0"/>
+    <geometry>
+      <mesh filename="file://$(find rov_description)/meshes/VerticalThrusterBeams_V7_v1__1__1.stl" scale="0.001 0.001 0.001"/>
+    </geometry>
+  </collision>
+</link>
+<link name="T200_v2__7__1">
+  <inertial>
+    <origin xyz="-0.041484995525996715 -0.026847398511978038 5.272863101965508e-06" rpy="0 0 0"/>
+    <mass value="0.15063623141000587"/>
+    <inertia ixx="0.000154" iyy="0.000156" izz="0.000141" ixy="-1.8e-05" iyz="-0.0" ixz="0.0"/>
+  </inertial>
+  <visual>
+    <origin xyz="0.26777 0.322691 -0.057622" rpy="0 0 0"/>
+    <geometry>
+      <mesh filename="file://$(find rov_description)/meshes/T200_v2__7__1.stl" scale="0.001 0.001 0.001"/>
+    </geometry>
+    <material name="silver"/>
+  </visual>
+  <collision>
+    <origin xyz="0.26777 0.322691 -0.057622" rpy="0 0 0"/>
+    <geometry>
+      <mesh filename="file://$(find rov_description)/meshes/T200_v2__7__1.stl" scale="0.001 0.001 0.001"/>
+    </geometry>
+  </collision>
+</link>
+<link name="T200_v2__1__1">
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